File: TapBeerFlowControl_hardware.kicad_pcb (KiCad board)
At the start: 2 copper layers, 58.2 x 62.6 mm, 22 parts, among them J1 12_VIN, J2 SENSOR, J3 SEL1, J4 SEL2, J5 SEL3, J6 VALVE_OUT, K1 JQC-3FC_T73_DC05V, Q1 BC547, SW1 SW_DIP_x01, U1 LM7805_TO220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

Commit message: adjust pending tasks in TODO file
Parts:
- J2: footprint Connector_JST:JST_EH_B3B-EH-A_1x03_P2.50mm_Vertical -> Connector_JST:JST_PH_B3B-PH-K_1x03_P2.00mm_Vertical
- J3, J4, J5: footprint Connector_JST:JST_EH_B2B-EH-A_1x02_P2.50mm_Vertical -> Connector_JST:JST_PH_B2B-PH-K_1x02_P2.00mm_Vertical
- Q1: footprint Package_TO_SOT_THT:TO-92_Inline -> Package_TO_SOT_THT:TO-92_HandSolder
- moved Q1 1.73 mm to (152.9, 59.0), turned to 0 degrees
- moved C2 1.70 mm to (125.4, 78.6)
- moved J2 0.94 mm to (113.9, 55.8)
- moved J3 0.91 mm to (113.4, 37.6)
- moved J5 0.72 mm to (113.6, 49.5)
- moved C1 0.66 mm to (126.1, 87.1)
- moved R1 0.52 mm to (119.0, 54.1)
Routing:
- net Net-(D2-A): track 18.8 -> 21.2 mm
- net +5V: track 68.1 -> 70.0 mm
- net /SEL1: track 8.19 -> 9.19 mm
- net /SEL3: track 6.47 -> 7.18 mm
- net Net-(J2-Pin_2): track 10.7 -> 10.2 mm
